File: Jocket_Split_LP/PCB/WristRest.kicad_pcb (KiCad board)
At the start: 2 copper layers, 132.7 x 54.8 mm, 0 parts

Commit message: Case Improvements
Other:
- board size 132.7 x 54.8 mm -> 134.7 x 77.9 mm
Changed lines of the file:
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@@
   (gr_line (start 97.45 142.65) (end 103.85 139.6) (layer "Edge.Cuts") (width 0.1))
   (gr_arc (start 222.69607 123.435293) (mid 201.767199 127.340242) (end 180.55 129.1) (layer "Edge.Cuts") (width 0.1))
-  (gr_arc (start 226.55 128.45) (mid 167.522342 176.983913) (end 95.675 150.95) (layer "Edge.Cuts") (width 0.1))
-  (gr_arc (start 222.69607 123.435293) (mid 226.383232 124.58989) (end 226.55 128.45) (layer "Edge.Cuts") (width 0.1))
+  (gr_arc (start 227.85 126.775) (mid 171.766332 200.130661) (end 93.725 150.775) (layer "Edge.Cuts") (width 0.1))
+  (gr_arc (start 222.69607 123.435293) (mid 226.062803 123.886355) (end 227.85 126.775) (layer "Edge.Cuts") (width 0.1))
   (gr_line (start 148.45 129.35) (end 180.55 129.1) (layer "Edge.Cuts") (width 0.1))
   (gr_arc (start 103.85 139.6) (mid 125.620271 132.170033) (end 148.45 129.35) (layer "Edge.Cuts") (width 0.1))
-  (gr_arc (start 95.675 150.95) (mid 94.473068 146.353163) (end 97.45 142.65) (layer "Edge.Cuts") (width 0.1))
+  (gr_arc (start 93.725 150.775) (mid 94.086781 146.029417) (end 97.45 142.65) (layer "Edge.Cuts") (width 0.1))
 )
